File: kicad/led_cube/led_cube.sch (KiCad schematic (older format))
At the start: 76 parts, among them U1 led_cube

Commit message: Added lots of stuff
Parts:
- removed LM1, LM10, LM11, LM12, LM13, LM14, LM15, LM16, LM17, LM18, LM19, LM2, LM20, LM21, LM22, LM23, LM24, LM25, LM26, LM27, LM28, LM29, LM3, LM30, LM31, LM32, LM34, LM35, LM36, LM37, LM38, LM39, LM4, LM40, LM41, LM42, LM43, LM44, LM45, LM46, LM47, LM48, LM49, LM5, LM50, LM51, LM52, LM53, LM54, LM55, LM56, LM57, LM58, LM59, LM6, LM60, LM61, LM62, LM63, LM64, LM7, LM8, LM9: LM, Resistor_THT:R_Axial_DIN0207_L6.3mm_D2.5mm_P7.62mm_Horizontal, symbol Device:R
- added A2: actual_arduino, footprints:nano, symbol MCU_Module:Arduino_Nano_v3.x
- added C1EX1, C1EX2, C1EX3, C1EX4, C1EX5, C1EX6, C1EX7, C2EX1, C2EX2, C2EX3, C2EX4, C2EX5, C2EX6, C2EX7: EX, Connector_PinHeader_2.54mm:PinHeader_1x01_P2.54mm_Vertical, symbol Connector:Conn_01x01_Female
- added Controller1, Controller2: controller, house_cube:15pin_controller, symbol house_cube:controller
- added QH'_EX1, plane1, plane2, plane3, plane4, plane5, plane6, plane7, plane8: (no value), Connector_PinHeader_2.54mm:PinHeader_1x01_P2.54mm_Vertical, symbol Connector:Conn_01x01_Female
- added R1, R10, R11, R12, R13, R14, R15, R16, R17, R18, R19, R2, R20, R21, R22, R23, R24, R25, R26, R27, R28, R29, R3, R30, R31, R32, R33, R34, R35, R36, R37, R38, R39, R4, R40, R41, R42, R43, R44, R45, R46, R47, R48, R49, R5, R50, R51, R52, R53, R54, R55, R56, R57, R58, R59, R6, R60, R61, R62, R63, R7, R8, R9: (no value), Resistor_THT:R_Axial_DIN0207_L6.3mm_D2.5mm_P7.62mm_Horizontal, symbol Device:R
- added _1, _2, _3, _4, _5, _6, _7, _8: _, house_cube:proto, symbol house_cube:_
- added fet1, fet2, fet3, fet4, fet5, fet6, fet7, fet8: gen_mosfet, house_cube:gen_fet, symbol house_cube:gen_mosfet
- added power_extern1: power, footprints:power, symbol Connector_Generic:Conn_01x02
- A1: value Arduino_Nano_v3.x -> arduino_buffer; footprint footprints:nano -> house_cube:nano_buffer
- R0: renamed from LM33; value LM -> (none)
Connections:
- net +5V: now also A1.30 (VIN), Controller1.2 (VCC), Controller2.2 (VCC), power_extern1.2 (Pin_2)
- net GND: now also A1.29 (GND), A1.4 (GND), Controller1.1 (GND), Controller2.1 (GND), fet1.3 (src), fet2.3 (src), fet3.3 (src), fet4.3 (src), fet5.3 (src), fet6.3 (src), fet7.3 (src), fet8.3 (src), power_extern1.1 (Pin_1); no longer SHIFT0.13 (~OE), SHIFT1.13 (~OE), SHIFT2.13 (~OE), SHIFT3.13 (~OE), SHIFT4.13 (~OE), SHIFT5.13 (~OE), SHIFT6.13 (~OE), SHIFT7.13 (~OE), SHIFT_PLANE1.13 (~OE)
- net led0: now also R0.2
- net led1: now also R1.2
- net led10: now also R10.2
- net led11: now also R11.2
- net led12: now also R12.2
- net led13: now also R13.2
- net led14: now also R14.2
- net led15: now also R15.2
- net led16: now also R16.2
- net led17: now also R17.2
- net led18: now also R18.2
- net led19: now also R19.2
- net led2: now also R2.2
- net led20: now also R20.2
- net led21: now also R21.2
- net led22: now also R22.2
- net led23: now also R23.2
- net led24: now also R24.2
- net led25: now also R25.2
- net led26: now also R26.2
- net led27: now also R27.2
- net led28: now also R28.2
- net led29: now also R29.2
- net led3: now also R3.2
- net led30: now also R30.2
- net led31: now also R31.2
- net led32: now also R32.2
- net led33: now also R33.2
- net led34: now also R34.2
- net led35: now also R35.2
- net led36: now also R36.2
- net led37: now also R37.2
- net led38: now also R38.2
- net led39: now also R39.2
- net led4: now also R4.2
- net led40: now also R40.2
- net led41: now also R41.2
- net led42: now also R42.2
- net led43: now also R43.2; no longer R0.1
- net led44: now also R44.2
- net led45: now also R45.2
- net led46: now also R46.2
- net led47: now also R47.2
- net led48: now also R48.2
- net led49: now also R49.2
- net led5: now also R5.2
- net led50: now also R50.2
- net led51: now also R51.2
- net led52: now also R52.2
- net led53: now also R53.2
- net led54: now also R54.2
- net led55: now also R55.2
- net led56: now also R56.2
- net led57: now also R57.2
- net led58: now also R58.2
- net led59: now also R59.2
- net led6: now also R6.2
- net led60: now also R60.2
- net led61: now also R61.2
- net led62: now also R62.2
- net led63: now also R63.2
- net led7: now also R7.2
- net led8: now also R8.2
- net led9: now also R9.2
- net plane1: now also fet1.2 (drn), plane1.1 (Pin_1); no longer SHIFT_PLANE1.1 (QB)
- net plane2: now also fet2.2 (drn), plane2.1 (Pin_1); no longer SHIFT_PLANE1.2 (QC)
- net plane3: now also fet3.2 (drn), plane3.1 (Pin_1); no longer SHIFT_PLANE1.3 (QD)
- net plane4: now also fet4.2 (drn), plane4.1 (Pin_1); no longer SHIFT_PLANE1.4 (QE)
- net plane5: now also fet5.2 (drn), plane5.1 (Pin_1); no longer SHIFT_PLANE1.5 (QF)
- net plane6: now also fet6.2 (drn), plane6.1 (Pin_1); no longer SHIFT_PLANE1.6 (QG)
- net plane7: now also fet7.2 (drn), plane7.1 (Pin_1); no longer SHIFT_PLANE1.7 (QH)
- net srclk: now also A1.16 (D13); no longer A1.7 (D4)
- net BUTTON_CLOCK: now reaches A1.10 (D7)
- net BUTTON_CLOCK: now also Controller1.3 (BUTTON_CLK), Controller2.3 (BUTTON_CLK)
- net BUTTON_LATCH: now reaches A1.11 (D8)
- net BUTTON_LATCH: now also Controller1.5 (BUTTON_LATCH), Controller2.5 (BUTTON_LATCH)
- net BUTTON_DATA: now reaches A1.12 (D9)
- net BUTTON_DATA: now also Controller1.4 (BUTTON_DATA), Controller2.4 (BUTTON_DATA)
- net data: now reaches A1.14 (D11)
- net data: now also SHIFT0.14 (SER)
- net JOY_V2: now reaches A1.23 (A4)
- net JOY_V2: now also Controller2.7 (A_JOY_VERT)
- net JOY_V1: now reaches A1.24 (A5)
- net JOY_V1: now also Controller1.7 (A_JOY_VERT)
- net JOY_H2: now reaches A1.25 (A6)
- net JOY_H2: now also Controller2.6 (A_JOY_HORZ)
- net JOY_H1: now reaches A1.26 (A7)
- net JOY_H1: now also Controller1.6 (A_JOY_HORZ)
- net BUTTON_WATCH2: now reaches A1.6 (D3)
- net BUTTON_WATCH2: now also Controller2.8 (BUTTON_WATCH)
- net at SHIFT7.9 (QH'): now also SHIFT_PLANE1.14 (SER); no longer SHIFT_PLANE1.9 (QH')
- net at U1.0 (row): now also R0.1
- net at U1.1 (row): now also R1.1
- net at U1.10 (row): now also R10.1
- net at U1.11 (row): now also R11.1
- net at U1.12 (row): now also R12.1
- net at U1.13 (row): now also R13.1
- net at U1.14 (row): now also R14.1
- net at U1.15 (row): now also R15.1
- net at U1.16 (row): now also R16.1
- net at U1.17 (row): now also R17.1
- net at U1.18 (row): now also R18.1
- net at U1.19 (row): now also R19.1
- net at U1.2 (row): now also R2.1
- net at U1.20 (row): now also R20.1
- net at U1.21 (row): now also R21.1
- net at U1.22 (row): now also R22.1
- net at U1.23 (row): now also R23.1
- net at U1.24 (row): now also R24.1
- net at U1.25 (row): now also R25.1
- net at U1.26 (row): now also R26.1
- net at U1.27 (row): now also R27.1
- net at U1.28 (row): now also R28.1
- net at U1.29 (row): now also R29.1
- net at U1.3 (row): now also R3.1
- net at U1.30 (row): now also R30.1
- net at U1.31 (row): now also R31.1
- net at U1.32 (row): now also R32.1
- net at U1.33 (row): now also R33.1
- net at U1.34 (row): now also R34.1
- net at U1.35 (row): now also R35.1
- net at U1.36 (row): now also R36.1
- net at U1.37 (row): now also R37.1
- net at U1.38 (row): now also R38.1
- net at U1.39 (row): now also R39.1
- net at U1.4 (row): now also R4.1
- net at U1.40 (row): now also R40.1
- net at U1.41 (row): now also R41.1
- net at U1.42 (row): now also R42.1
- net at U1.43 (row): now also R43.1
- net at U1.44 (row): now also R44.1
- net at U1.45 (row): now also R45.1
- net at U1.46 (row): now also R46.1
- net at U1.47 (row): now also R47.1
- net at U1.48 (row): now also R48.1
- net at U1.49 (row): now also R49.1
- net at U1.5 (row): now also R5.1
- net at U1.50 (row): now also R50.1
- net at U1.51 (row): now also R51.1
- net at U1.52 (row): now also R52.1
- net at U1.53 (row): now also R53.1
- net at U1.54 (row): now also R54.1
- net at U1.55 (row): now also R55.1
- net at U1.56 (row): now also R56.1
- net at U1.57 (row): now also R57.1
- net at U1.58 (row): now also R58.1
- net at U1.59 (row): now also R59.1
- net at U1.6 (row): now also R6.1
- net at U1.60 (row): now also R60.1
- net at U1.61 (row): now also R61.1
- net at U1.62 (row): now also R62.1
- net at U1.63 (row): now also R63.1; no longer R0.2
- net at U1.7 (row): now also R7.1
- net at U1.8 (row): now also R8.1
- net at U1.9 (row): now also R9.1
- net d6 renamed BUTTON_WATCH1
- net BUTTON_WATCH1: now also Controller1.8 (BUTTON_WATCH); no longer SHIFT0.14 (SER)
- net plane0 renamed pg0
- net pg0: now also fet1.1 (gt)
- new net: QH'_EX1.1 (Pin_1), SHIFT_PLANE1.9 (QH')
- new net: C1EX2.1 (Pin_1), Controller1.10 (EXTRA_1)
- new net: C1EX3.1 (Pin_1), Controller1.11 (EXTRA_2)
- new net: C1EX4.1 (Pin_1), Controller1.12 (EXTRA_3)
- new net: C1EX5.1 (Pin_1), Controller1.13 (EXTRA_4)
- new net: C1EX6.1 (Pin_1), Controller1.14 (EXTRA_5)
- new net: C1EX7.1 (Pin_1), Controller1.15 (EXTRA_7)
- new net: C1EX1.1 (Pin_1), Controller1.9 (EXTRA_0)
- new net: C2EX2.1 (Pin_1), Controller2.10 (EXTRA_1)
- new net: C2EX3.1 (Pin_1), Controller2.11 (EXTRA_2)
- new net: C2EX4.1 (Pin_1), Controller2.12 (EXTRA_3)
- new net: C2EX5.1 (Pin_1), Controller2.13 (EXTRA_4)
- new net: C2EX6.1 (Pin_1), Controller2.14 (EXTRA_5)
- new net: C2EX7.1 (Pin_1), Controller2.15 (EXTRA_7)
- new net: C2EX1.1 (Pin_1), Controller2.9 (EXTRA_0)
- new net output_enable: A1.7 (D4), SHIFT0.13 (~OE), SHIFT1.13 (~OE), SHIFT2.13 (~OE), SHIFT3.13 (~OE), SHIFT4.13 (~OE), SHIFT5.13 (~OE), SHIFT6.13 (~OE), SHIFT7.13 (~OE), SHIFT_PLANE1.13 (~OE)
- new net pg1: SHIFT_PLANE1.1 (QB), fet2.1 (gt)
- new net pg2: SHIFT_PLANE1.2 (QC), fet3.1 (gt)
- new net pg3: SHIFT_PLANE1.3 (QD), fet4.1 (gt)
- new net pg4: SHIFT_PLANE1.4 (QE), fet5.1 (gt)
- new net pg5: SHIFT_PLANE1.5 (QF), fet6.1 (gt)
- new net pg6: SHIFT_PLANE1.6 (QG), fet7.1 (gt)
- new net pg7: SHIFT_PLANE1.7 (QH), fet8.1 (gt)
- new net plane8: fet8.2 (drn), plane8.1 (Pin_1)
- no-connect marks 0 -> 136
Other:
- moved on the sheet: A1, R0, SHIFT0, SHIFT1, SHIFT2, SHIFT3, SHIFT4, SHIFT5, SHIFT6, SHIFT7, SHIFT_PLANE1, power1
